Commit message: add camera and publish image, no correct point cloud

File: src/franka_ros2/franka_description/robots/common/dual_robot.xacro (robot description, xacro)
@@ -35,5 +35,7 @@
                       fake_sensor_commands2:=false
                       gazebo_effort1:=true
-                      gazebo_effort2:=true">
+                      gazebo_effort2:=true
+                      camera1:=true
+                      camera2:=true">
     <xacro:include filename="$(find franka_description)/robots/common/utils.xacro" />
     <xacro:include filename="$(find franka_description)/robots/common/dual_arm.xacro" />
@@ -68,5 +70,5 @@
     <xacro:include filename="$(find franka_description)/end_effectors/common/dual_hand.xacro"/>
     <xacro:include filename="$(find franka_description)/end_effectors/common/dual_utils.xacro" />
-    <!-- <xacro:include filename="$(find franka_description)/end_effectors/franka_hand/dual_hand_arguments.xacro" /> -->
+   <xacro:if value="${hand1}">
     <xacro:franka_hand
       connected_to="$(arg arm_id1)_link8"
@@ -81,4 +83,12 @@
       with_sc="${with_sc1}"
     />
+    <xacro:if value="${camera1}">
+      <xacro:include filename="$(find realsense_ros_gazebo)/xacro/fr3_camera.xacro"/>
+      <xacro:realsense_d435 sensor_name="fr3_camera" parent_link="${arm_id1}_hand" rate="10">
+        <origin rpy="3.14 0 0" xyz="0.03 0.0 0.046369403"/>
+      </xacro:realsense_d435>
+    </xacro:if>
+   </xacro:if>
+   <xacro:if value="${hand2}">
     <xacro:franka_hand
       connected_to="$(arg arm_id2)_link8"
@@ -93,4 +103,11 @@
       with_sc="${with_sc2}"
     />
+    <xacro:if value="${camera2}">
+      <xacro:include filename="$(find realsense_ros_gazebo)/xacro/fp3_camera.xacro"/>
+      <xacro:realsense_d435 sensor_name="${arm_id2}_camera" parent_link="${arm_id2}_hand" rate="10">
+        <origin rpy="3.14 0 0" xyz="0.03 0.0 0.046369403"/>
+      </xacro:realsense_d435>
+    </xacro:if>
+   </xacro:if>
     <xacro:if value="${gazebo1}">
       <xacro:gazebo-joint joint="${arm_id1}_joint1" transmission="hardware_interface/PositionJointInterface" />

File: src/franka_ros2/franka_description/robots/dual_arm/dual_arm.urdf.xacro (robot description, xacro)
@@ -38,4 +38,6 @@
   <xacro:arg name="parent1" default="world" />
   <xacro:arg name="parent2" default="fr3_link0" />
+  <xacro:arg name="camera1" default="true" />
+  <xacro:arg name="camera2" default="true" />
   <xacro:franka_robot arm_id1="$(arg arm_id1)"
                       arm_id2="$(arg arm_id2)"
@@ -71,5 +73,7 @@
                       rpy2="$(arg rpy2)"
                       parent1="$(arg parent1)"
-                      parent2="$(arg parent2)">
+                      parent2="$(arg parent2)"
+                      camera1="$(arg camera1)"
+                      camera2="$(arg camera2)">
   </xacro:franka_robot>
 </robot>
